Commit message: end project

File: description/robot.urdf.xacro (robot description, xacro)
@@ -4,3 +4,5 @@
   <xacro:include filename="gazebo_control.xacro" />
   <xacro:include filename="robot_core.xacro" />
+  <xacro:include filename="camera.xacro" />
+  <xacro:include filename="lidar.xacro" />
 </robot>

File: description/robot_core.xacro (robot description, xacro)
@@ -1,4 +1,4 @@
 <?xml version="1.0"?>
-<robot xmlns:xacro="http://www.ros.org/wiki/xacro">
+<robot name="arty_bot" xmlns:xacro="http://www.ros.org/wiki/xacro">
 <xacro:include filename="inertial_macros.xacro" />
 <material name="white">
@@ -13,4 +13,7 @@
 <material name="black">
     <color rgba="0 0 0 1"/>
+</material>
+<material name="red">
+    <color rgba="1 0 0 1"/>
 </material>
 <link name="base_link">
